Commit message: Added launchfile to test odometry. Changed rviz and urdf files to comply

File: autonomous_car/urdf/robotCar.urdf (robot description, URDF)
Before this commit: robot myfirst, 5 links, 4 joints
Links:
- link body_link: geometry visual box size=3.332 1.28 1.7
Joints:
- joint body_to_back_left_wheel: origin xyz=-0.64 0 0 rpy=0 -1.57075 0 -> xyz=0 -0.64 0 rpy=-1.57075 0 0
- joint body_to_back_right_wheel: origin xyz=0.64 0 0 rpy=0 -1.57075 0 -> xyz=0 0.64 0 rpy=-1.57075 0 0
- joint body_to_steering_point: origin xyz=0 2.2 0 rpy=0 -1.57075 0 -> xyz=2.2 0 0
- joint steering_point_to_front_wheel: origin (none) -> rpy=-1.57075 0 0

Commit message: Odometry uses steering. Add proportional control.

File: autonomous_car/urdf/robotCar.urdf (robot description, URDF)
Before this commit: robot myfirst, 5 links, 4 joints
Joints:
- joint body_to_steering_point: axis 1 0 0 -> 0 0 1

Commit message: move_base makes trajectory plan however car does not receive correct commands

File: autonomous_car/urdf/robotCar.urdf (robot description, URDF)
Before this commit: robot myfirst, 5 links, 4 joints
Links:
- removed link body_link
- added link base_footprint
- added link base_link; visual box size=3.332 1.28 1.5
- link back_left_wheel: geometry visual cylinder length=0.114 radius=0.256
- link back_right_wheel: geometry visual cylinder length=0.114 radius=0.256
- link front_wheel: geometry visual cylinder length=0.114 radius=0.256
Joints:
- removed joint body_to_back_left_wheel
- removed joint body_to_back_right_wheel
- added joint base_joint: type fixed, parent base_footprint, child base_link, origin xyz=0 0 0 rpy=0 0 0
- added joint base_to_back_left_wheel: type continuous, parent base_link, child back_left_wheel, origin xyz=0 -0.64 0 rpy=-1.57075 0 0, axis 0 0 1
- added joint base_to_back_right_wheel: type continuous, parent base_link, child back_right_wheel, origin xyz=0 0.64 0 rpy=-1.57075 0 0, axis 0 0 1
- joint body_to_steering_point: parent body_link -> base_link

File: robotics_lab2/urdf/aut_car.urdf (robot description, URDF)
Before this commit: robot car_model, 5 links, 4 joints
Links:
- added link steering_point
Joints:
- removed joint front_wheel_joint
- added joint base_to_steering_point: type continuous, parent base_link, child steering_point, origin xyz=2.2 0 0, axis 0 0 1
- added joint steering_point_to_front_wheel: type continuous, parent steering_point, child front_wheel_link, origin rpy=-1.57075 0 0, axis 0 0 1
- joint back_wheel_left_joint: origin xyz=0.0 0.64 0 rpy=-1.57075 0 0 -> xyz=0.0 0.64 0 rpy=1.57075 0 0

File: robotics_lab2/urdf/robotCar.urdf (robot description, URDF)
Before this commit: robot autonomous_car, 5 links, 4 joints
Links:
- removed link body_link
- added link base_footprint
- added link base_link; visual box size=3.332 1.28 1.5
- link back_left_wheel: geometry visual cylinder length=0.114 radius=0.256
- link back_right_wheel: geometry visual cylinder length=0.114 radius=0.256
- link front_wheel: geometry visual cylinder length=0.114 radius=0.256
Joints:
- removed joint body_to_back_left_wheel
- removed joint body_to_back_right_wheel
- added joint base_joint: type fixed, parent base_footprint, child base_link, origin xyz=220 183.41 0 rpy=0 0 1.57075
- added joint base_to_back_left_wheel: type continuous, parent base_link, child back_left_wheel, origin xyz=0 -0.64 0 rpy=1.57075 0 0, axis 0 0 1
- added joint base_to_back_right_wheel: type continuous, parent base_link, child back_right_wheel, origin xyz=0 0.64 0 rpy=-1.57075 0 0, axis 0 0 1
- joint body_to_steering_point: parent body_link -> base_link
